File: pcb/bioterio_v01.kicad_pcb (KiCad board)
At the start: 2 copper layers, 47 x 101.6 mm, 20 parts, among them J1 12V_in, J2 BME280_1, J3 Relais_Out, J4 12V_out, J5 LED_Strip_Out, J6 BME280_2, J7 Disp_Out, U1 L7805, U2 voltage_conv, U3 WeMos_D1_mini

Commit message: getting gerber and such
Parts:
- removed J5: LED_Strip_Out, TerminalBlock_Phoenix:TerminalBlock_Phoenix_MKDS-1,5-4-5.08_1x04_P5.08mm_Horizontal
- added REF**: h1, MountingHole:MountingHole_3.2mm_M3_DIN965, F.Cu at (130.8, 40.6)
- added REF**: h1, MountingHole:MountingHole_3.2mm_M3_DIN965, F.Cu at (99.1, 34.3)
- added REF**: h1, MountingHole:MountingHole_3.2mm_M3_DIN965, F.Cu at (99.1, 100.3)
- added REF**: h1, MountingHole:MountingHole_3.2mm_M3_DIN965, F.Cu at (139.7, 115.6)
- added ctrl: LED_Strip_Out, TerminalBlock_Phoenix:TerminalBlock_Phoenix_MKDS-1,5-4-5.08_1x04_P5.08mm_Horizontal, F.Cu at (138.4, 31.8)
- J1: value 12V_in -> +12V
- J4: value 12V_out -> +12V
- renumbered J6 to disp, J7 to sens_1, J2 to sens_2
Other:
- board size 47 x 101.6 mm -> 47 x 95.2 mm
- board text added: "+5V"
- board text added: "3.3v"
- board text added: "5v"
- board text added: "SCL"
- board text added: "SDA"
- board text added: "bioterio v01 05/2020"
- board text added: "ctrl"
- board text added: "r0oland corona_times 2020"
